File: rsp.02_EM#001.sch (KiCad schematic (older format))
At the start: 447 parts

Commit message: Update for S-MacBookPro
Parts:
- removed C?: 1u, Capacitors_SMD:C_0603, symbol Device:C_Small
- removed C?: 10u, Capacitors_SMD:C_0603, symbol rsp.02_EM#001-rescue:C_Small-RSP-01P_FM-rescue-RSP-02P_BBM-rescue-rsp.02_BBM_mo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
- removed C?: 10u, Capacitors_THT:C_Rect_L4.6mm_W4.6mm_P2.50mm_MKS02_FKP02, symbol rsp.02_EM#001-rescue:C_Small-RSP-01P_FM-rescue-RSP-02P_BBM-rescue-rsp.02_BBM_mo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
- removed H?: MountingHole_Pad, Mounting_Holes:MountingHole_3.2mm_M3_Pad, symbol Mechanical:MountingHole_Pad
- removed H? (x3): MountingHole, Mounting_Holes:MountingHole_3.2mm_M3, symbol Mechanical:MountingHole
- removed JP?: Jumper, Connectors:GS2, symbol mypartsLib:Jumper_NO_Small-Device
- removed L?: 3.3uH, Inductors_SMD:L_Taiyo-Yuden_NR-50xx_HandSoldering, symbol rsp.02_EM#001-rescue:INDUCTOR_SMALL-RSP-01P_FM-rescue-RSP-02P_BBM-rescue-rsp.02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
- removed Q? (x2): BC857BS, TO_SOT_Packages_SMD:SOT-363_SC-70-6, symbol Transistor_BJT:BC857BS
- removed R?: 910k, Resistors_SMD:R_0603, symbol mypartsLib:R-RSP-00P
- removed R?: 1M, Resistors_SMD:R_0603, symbol Device:R
- removed TP? (x3): TestPoint, Measurement_Points:Measurement_Point_Round-SMD-Pad_Small, symbol Connector:TestPoint
- added C?: 1u, Capacitors_SMD:C_0603, symbol Device:C_Small
- added C?: 10u, Capacitors_SMD:C_0603, symbol Device:C_Small
- added C?: 10u, Capacitors_THT:C_Rect_L4.6mm_W4.6mm_P2.50mm_MKS02_FKP02, symbol Device:C_Small
- added JP?: Jumper, Connectors:GS2, symbol mypartsLib:Jumper_NO_Small-Device
- added L?: 3.3uH, Inductors_SMD:L_Taiyo-Yuden_NR-50xx_HandSoldering, symbol pspice:INDUCTOR
- added Q? (x2): BC857BS, TO_SOT_Packages_SMD:SOT-363_SC-70-6, symbol Transistor_BJT:BC857BS
- added R?: 910k, Resistors_SMD:R_0603, symbol mypartsLib:R-RSP-00P
- added R?: 1M, Resistors_SMD:R_0603, symbol Device:R
- added TP? (x3): TestPoint, Measurement_Points:Measurement_Point_Round-SMD-Pad_Small, symbol Connector:TestPoint
- C? (x28): symbol rsp.02_EM#001-rescue:C_Small-RSP-01P_FM-rescue-RSP-02P_BBM-rescue-rsp.02_BBM_modules##001-rescue-rsp.02_BBM_Modules##00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 -> Device:C_Small
- JP? (x5): symbol mypartsLib:Jumper_NC_Small-Device -> mypartsLib:Jumper_NO_Small-Device
- L? (x4): symbol rsp.02_EM#001-rescue:INDUCTOR_SMALL-RSP-01P_FM-rescue-RSP-02P_BBM-rescue-rsp.02_BBM_modules##001-rescue-rsp.02_BBM_Modu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 -> pspice:INDUCTOR
- Q?: symbol Katsunori:IRFHM9331PbF -> mypartsLib:IRFHM9331PbF
- R? (x12): symbol rsp.02_EM#001-rescue:R-RESCUE-RS-00P_TestBoard1-RSP-01P_FM-rescue-RSP-02P_BBM-rescue-rsp.02_BBM_modules##001-rescue-rsp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 -> mypartsLib:R-RSP-00P
- U? (x5): symbol KiCad:LTC3130 -> mypartsLib:LTC3130-compact
Connections:
- net labels removed: Earth
- wire segments 925 -> 921
Other:
- note removed: "1-point GND to \n Satellite body structure.\nNo other GND pts shall be \n grounded to the body."
- note removed: "1-point connection \namong all type of grounds."

Commit message: Update from S-MacBookPro
Parts:
- removed R?: 1M, Resistors_SMD:R_0603, symbol Device:R
- added R?: 1M, Resistors_SMD:R_0603, symbol Device:R
Changed lines of the file:
@@
 $Descr A3 16535 11693
 encoding utf-8
-Sheet 18 20
+Sheet 18 33
 Title "RSP-02 PCU EM"
 Date "2021-02-27"
@@
 $Comp
 L Device:R R?
-U 1 1 62DD8487
+U 1 1 6051F955
 P 6050 1850
 F 0 "R?" V 6150 1750 50  0000 L CNN
