File: rsp02_Power_Circuit_EM_v1_0.sch (KiCad schematic (older format))
At the start: 35 parts, among them J1 Conn_01x02, J10 Conn_01x02, J11 Conn_01x02, J12 Conn_01x02, J13 Conn_01x02, J14 Conn_01x02, J15 Conn_01x10, J16 Conn_01x10, J2 Conn_01x02, J3 Conn_01x02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

Commit message: Update for S-MacBookPro
Parts:
- added H?: MountingHole_Pad, Mounting_Holes:MountingHole_3.2mm_M3_Pad, symbol Mechanical:MountingHole_Pad
- added H? (x3): MountingHole, Mounting_Holes:MountingHole_3.2mm_M3, symbol Mechanical:MountingHole
- added JP? (x9): Jumper, Connectors:GS2, symbol mypartsLib:Jumper_NO_Small-Device
- added JP?: Jumper_NC_Small-Device, symbol mypartsLib:Jumper_NC_Small-Device
Connections:
- net GNDA renamed Earth
- net Earth: now also H?.1
- new net PV1(+): JP?.1
- new net PV1(-): JP?.1, JP?.1, JP?.1, JP?.1
- new net PV2(+): JP?.1
- new net PV3(+): JP?.1
- new net PV4(+): JP?.1
- new net PV5(+): JP?.1
- new net PVC1_Ideal_Diode/Anode: JP?.2
- new net PVC1_MPPT_Circuit/VOUT: JP?.1
Other:
- note added: "1-point GND to \n Satellite body structure.\nNo other GND pts shall be \n grounded to the body."
- note added: "1-point connection \namong all type of grounds."
- note added: "OCP : Deactive"
- note added: "PCU100 : PVC#1 MPPT Circuit"
- note added: "PCU120 : PVC#2 MPPT Circuit"
- note added: "PCU140 : PVC#3 MPPT Circuit"
- note added: "PCU160 : PVC#4 MPPT Circuit"
- note added: "PCU180 : PVC#5 MPPT Circuit"
- note added: "PVC#1"
- note added: "PVC#2"
- note added: "PVC#3"
- note added: "PVC#4"
- note added: "PVC#5"
- note removed: "OCP : \nDeactive"
- moved on the sheet: R1, R2, R3

Commit message: Update from S-MacBookPro
Parts:
- removed JP? (x9): Jumper, Connectors:GS2, symbol mypartsLib:Jumper_NO_Small-Device
- added JP? (x19): Jumper_NC_Small-Device, symbol mypartsLib:Jumper_NC_Small-Device
Connections:
- net PV1(+): now also JP?.1
- net PV2(+): now also JP?.1
- net PV3(+): now also JP?.1
- net PV4(+): now also JP?.1
- net PV5(+): now also JP?.1
- net PVC1_Ideal_Diode/Cathode: now also JP?.1
- net PVC1_MPPT_Circuit/VOUT renamed PVC1_MPPT/VOUT
- new net PVC1_CS/OUTPUT: JP?.1
- new net PVC1_MPPT/PVIN: JP?.2
- new net PVC2_CS/OUTPUT: JP?.1
- new net PVC2_Ideal_Diode/Anode: JP?.2
- new net PVC2_Ideal_Diode/Cathode: JP?.1
- new net PVC2_MPPT/PVIN: JP?.2
- new net PVC2_MPPT/VOUT: JP?.1
- new net PVC3_CS/OUTPUT: JP?.1
- new net PVC3_Ideal_Diode/Anode: JP?.2
- new net PVC3_Ideal_Diode/Cathode: JP?.1
- new net PVC3_MPPT/PVIN: JP?.2
- new net PVC3_MPPT/VOUT: JP?.1
- new net PVC4_CS/OUTPUT: JP?.1
- new net PVC4_Ideal_Diode/Anode: JP?.2
- new net PVC4_Ideal_Diode/Cathode: JP?.1
- new net PVC4_MPPT/PVIN: JP?.2
- new net PVC4_MPPT/VOUT: JP?.1
- new net PVC5_CS/OUTPUT: JP?.1
- new net PVC5_Ideal_Diode/Anode: JP?.2
- new net PVC5_Ideal_Diode/Cathode: JP?.1
- new net PVC5_MPPT/PVIN: JP?.2
- new net PVC5_MPPT/VOUT: JP?.1
- new net Vmpp: JP?.2, JP?.2, JP?.2, JP?.2, JP?.2
- new net Vpvc1: JP?.2
- new net Vpvc2: JP?.2
- new net Vpvc3: JP?.2
- new net Vpvc4: JP?.2
- new net Vpvc5: JP?.2
Other:
- note added: "1-point connection between\nanalong GND and BAT GND."
- note added: "High-side \nDeployment \nSwitch#1"
- note added: "High-side\nDeployment\nSwitch#2"
- note added: "Low-side\nDeployment\nSwitch"
- note added: "MPPT"
- moved on the sheet: H?, JP?, R1, R10, R11, R12, R13, R14, R15, R16, R17, R18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
