File: rsp02_module_CS_PV.sch (KiCad schematic (older format))
At the start: 5 parts, among them IC14 INA199A1DCKT_v2

Commit message: Update from S-MacBookPro
Parts:
- added C?: 0.1u, Capacitor_SMD:C_0603_1608Metric, symbol Device:C
- added JP?: Jumper_NO_Small-Device, symbol mypartsLib:Jumper_NO_Small-Device
- added JP?: Jumper_NC_Small-Device, symbol mypartsLib:Jumper_NC_Small-Device
Connections:
- net GND: now also C?.2
- net INPUT: now also JP?.1; no longer C26.1, IC14.3 (V+)
- new net: C26.1, C?.1, IC14.3 (V+), JP?.2, JP?.2
- new net +3V3: JP?.1
Other:
- moved on the sheet: C26
Changed lines of the file:
@@
 $Descr A4 11693 8268
 encoding utf-8
-Sheet 17 33
+Sheet 20 33
 Title "rsp02_module_Current Sense_3_3V"
 Date "2020-12-07"
@@
 AR Path="/5FD18C31/5FD0FFD7" Ref="R108"  Part="1"
 AR Path="/5FD18BF5/5FD0FFD7" Ref="R111"  Part="1"
-F 0 "R117" V 5490 2500 50  0000 C CNN
+AR Path="/6051F923/5FD0FFD7" Ref="R?"  Part="1"
+AR Path="/60C25BD4/5FD0FFD7" Ref="R?"  Part="1"
+AR Path="/60C51ADC/5FD0FFD7" Ref="R?"  Part="1"
+AR Path="/60C74F70/5FD0FFD7" Ref="R?"  Part="1"
+AR Path="/60C9EA51/5FD0FFD7" Ref="R?"  Part="1"
+F 0 "R?" V 5490 2500 50  0000 C CNN
 F 1 "0.02" V 5660 2500 50  0000 C CNN
 F 2 "Resistor_SMD:R_2512_6332Metric" V 5500 2500 50  0001 C CNN
@@
 AR Path="/5FD18C31/5FCF83F6" Ref="R106"  Part="1"
 AR Path="/5FD18BF5/5FCF83F6" Ref="R109"  Part="1"
-F 0 "R115" V 4830 4450 50  0000 C CNN
+AR Path="/6051F923/5FCF83F6" Ref="R?"  Part="1"
+AR Path="/60C25BD4/5FCF83F6" Ref="R?"  Part="1"
+AR Path="/60C51ADC/5FCF83F6" Ref="R?"  Part="1"
+AR Path="/60C74F70/5FCF83F6" Ref="R?"  Part="1"
+AR Path="/60C9EA51/5FCF83F6" Ref="R?"  Part="1"
+F 0 "R?" V 4830 4450 50  0000 C CNN
 F 1 "0" V 4750 4340 50  0000 C CNN
 F 2 "Resistor_SMD:R_0603_1608Metric" V 4680 4340 50  0001 C CNN
@@
 AR Path="/5FD18C31/5FCF83F7" Ref="R107"  Part="1"
 AR Path="/5FD18BF5/5FCF83F7" Ref="R110"  Part="1"
-F 0 "R116" V 4840 4640 50  0000 C CNN
+AR Path="/6051F923/5FCF83F7" Ref="R?"  Part="1"
+AR Path="/60C25BD4/5FCF83F7" Ref="R?"  Part="1"
+AR Path="/60C51ADC/5FCF83F7" Ref="R?"  Part="1"
+AR Path="/60C74F70/5FCF83F7" Ref="R?"  Part="1"
+AR Path="/60C9EA51/5FCF83F7" Ref="R?"  Part="1"
+F 0 "R?" V 4840 4640 50  0000 C CNN
 F 1 "0" V 4750 4540 50  0000 C CNN
 F 2 "Resistor_SMD:R_0603_1608Metric" V 4680 4540 50  0001 C CNN
@@
 AR Path="/5FD18C31/5FCF83F8" Ref="IC11"  Part="1"
 AR Path="/5FD18BF5/5FCF83F8" Ref="IC12"  Part="1"
-F 0 "IC14" H 6100 5040 50  0000 C CNN
+AR Path="/6051F923/5FCF83F8" Ref="IC?"  Part="1"
+AR Path="/60C25BD4/5FCF83F8" Ref="IC?"  Part="1"
+AR Path="/60C51ADC/5FCF83F8" Ref="IC?"  Part="1"
+AR Path="/60C74F70/5FCF83F8" Ref="IC?"  Part="1"
+AR Path="/60C9EA51/5FCF83F8" Ref="IC?"  Part="1"
+F 0 "IC?" H 6100 5040 50  0000 C CNN
 F 1 "INA199A1DCKT_v2" H 6370 4950 50  0000 C CNN
 F 2 "Package_TO_SOT_SMD:SOT-363_SC-70-6" H 7120 4480 50  0001 L CNN
@@
 L Device:C C26
 U 1 1 5FD23316
-P 6370 3290
+P 6370 3320
 AR Path="/5FD18B52/5FD23316" Ref="C26"  Part="1"
 AR Path="/5FD18D07/5FD23316" Ref="C19"  Part="1"
@@
 AR Path="/5FD18C31/5FD23316" Ref="C23"  Part="1"
 AR Path="/5FD18BF5/5FD23316" Ref="C24"  Part="1"
-F 0 "C26" H 6485 3336 50  0000 L CNN
-F 1 "0.1u" H 6485 3245 50  0000 L CNN
-F 2 "Capacitor_SMD:C_0603_1608Metric" H 6408 3140 50  0001 C CNN
-F 3 "~" H 6370 3290 50  0001 C CNN
-	1    6370 3290
+AR Path="/6051F923/5FD23316" Ref="C?"  Part="1"
+AR Path="/60C25BD4/5FD23316" Ref="C?"  Part="1"
+AR Path="/60C51ADC/5FD23316" Ref="C?"  Part="1"
+AR Path="/60C74F70/5FD23316" Ref="C?"  Part="1"
+AR Path="/60C9EA51/5FD23316" Ref="C?"  Part="1"
+F 0 "C?" H 6485 3366 50  0000 L CNN
+F 1 "0.1u" H 6485 3275 50  0000 L CNN
+F 2 "Capacitor_SMD:C_0603_1608Metric" H 6408 3170 50  0001 C CNN
+F 3 "~" H 6370 3320 50  0001 C CNN
+	1    6370 3320
 	1    0    0    -1
 $EndComp
 Text HLabel 6270 3570 0    50   Input ~ 0
 GND
-Text HLabel 5470 3100 0    50   Input ~ 0
+Text HLabel 5200 3100 0    50   Input ~ 0
 INPUT
 Wire Wire Line
@@
 	6270 3570 6370 3570
 Wire Wire Line
-	6370 3140 6370 3100
-Wire Wire Line
-	6370 3100 5870 3100
+	6370 3170 6370 3100
+Wire Wire Line
+	6370 3570 6370 3470
+Wire Wire Line
+	5870 3100 5870 3760
+Text HLabel 5200 3350 0    50   Input ~ 0
++3V3
+$Comp
+L mypartsLib:Jumper_NO_Small-Device JP?
+U 1 1 60626F2A
+P 5500 3350
+AR Path="/6051F923/60626F2A" Ref="JP?"  Part="1"
+AR Path="/60C25BD4/60626F2A" Ref="JP?"  Part="1"
+AR Path="/60C51ADC/60626F2A" Ref="JP?"  Part="1"
+AR Path="/60C74F70/60626F2A" Ref="JP?"  Part="1"
+AR Path="/60C9EA51/60626F2A" Ref="JP?"  Part="1"
+F 0 "JP?" H 5500 3443 50  0000 C CNN
+F 1 "Jumper_NO_Small-Device" H 5500 3444 50  0001 C CNN
+F 2 "" H 5500 3350 50  0001 C CNN
+F 3 "" H 5500 3350 50  0001 C CNN
+	1    5500 3350
+	1    0    0    -1
+$EndComp
+$Comp
+L mypartsLib:Jumper_NC_Small-Device JP?
+U 1 1 60628634
+P 5500 3100
+AR Path="/6051F923/60628634" Ref="JP?"  Part="1"
+AR Path="/60C25BD4/60628634" Ref="JP?"  Part="1"
+AR Path="/60C51ADC/60628634" Ref="JP?"  Part="1"
+AR Path="/60C74F70/60628634" Ref="JP?"  Part="1"
+AR Path="/60C9EA51/60628634" Ref="JP?"  Part="1"
+F 0 "JP?" H 5500 3221 50  0000 C CNN
+F 1 "Jumper_NC_Small-Device" H 5500 3221 50  0001 C CNN
+F 2 "" H 5500 3100 50  0001 C CNN
+F 3 "" H 5500 3100 50  0001 C CNN
+	1    5500 3100
+	1    0    0    -1
+$EndComp
+Wire Wire Line
+	5600 3100 5800 3100
 Connection ~ 5870 3100
 Wire Wire Line
-	6370 3570 6370 3440
-Wire Wire Line
-	5470 3100 5870 3100
-Wire Wire Line
-	5870 3100 5870 3760
+	5600 3350 5800 3350
+Wire Wire Line
+	5800 3350 5800 3100
+Connection ~ 5800 3100
+Wire Wire Line
+	5800 3100 5870 3100
+Wire Wire Line
+	5400 3100 5200 3100
+Wire Wire Line
+	5200 3350 5400 3350
+$Comp
+L Device:C C?
+U 1 1 60630078
+P 6750 3320
+AR Path="/5FD18B52/60630078" Ref="C?"  Part="1"
+AR Path="/5FD18D07/60630078" Ref="C?"  Part="1"
+AR Path="/5FD18CD4/60630078" Ref="C?"  Part="1"
+AR Path="/5FD18CAB/60630078" Ref="C?"  Part="1"
+AR Path="/5FD18C72/60630078" Ref="C?"  Part="1"
+AR Path="/5FD18C31/60630078" Ref="C?"  Part="1"
+AR Path="/5FD18BF5/60630078" Ref="C?"  Part="1"
+AR Path="/6051F923/60630078" Ref="C?"  Part="1"
+AR Path="/60C25BD4/60630078" Ref="C?"  Part="1"
+AR Path="/60C51ADC/60630078" Ref="C?"  Part="1"
+AR Path="/60C74F70/60630078" Ref="C?"  Part="1"
+AR Path="/60C9EA51/60630078" Ref="C?"  Part="1"
+F 0 "C?" H 6865 3366 50  0000 L CNN
+F 1 "0.1u" H 6865 3275 50  0000 L CNN
+F 2 "Capacitor_SMD:C_0603_1608Metric" H 6788 3170 50  0001 C CNN
+F 3 "~" H 6750 3320 50  0001 C CNN
+	1    6750 3320
+	1    0    0    -1
+$EndComp
+Wire Wire Line
+	6750 3170 6750 3100
+Wire Wire Line
+	5870 3100 6370 3100
+Connection ~ 6370 3100
+Wire Wire Line
+	6370 3100 6750 3100
+Wire Wire Line
+	6370 3570 6750 3570
+Wire Wire Line
+	6750 3470 6750 3570
+Connection ~ 6370 3570
 $EndSCHEMATC
