File: rsp02_module_Ideal_Diode.sch (KiCad schematic (older format))
At the start: 7 parts

Commit message: Update from S-MacBookPro
Parts:
- removed Q?: IRFHM9331PbF, KiCad:PQFN-8-3x3mm_Pitch0.65mm, symbol mypartsLib:IRFHM9331PbF
- added Q?: IRFHM9331PbF, KiCad:PQFN-8-3x3mm_Pitch0.65mm, symbol mypartsLib:IRFHM9331PbF
Connections:
- net Anode: now also Q?.5 (D)
- net Cathode: now also Q?.1 (S)
- net at Q?.3 (C2), R?.2: now also Q?.4 (G)
Changed lines of the file:
@@
 $Descr A4 11693 8268
 encoding utf-8
-Sheet 19 20
+Sheet 30 33
 Title "RSP-02 PCU EM"
 Date "2021-03-15"
@@
 U 1 1 5F4AC996
 P 5350 4000
+AR Path="/60A4AB90/5F4AC996" Ref="Q?"  Part="1"
+AR Path="/60C25BC1/5F4AC996" Ref="Q?"  Part="1"
+AR Path="/60C51AC9/5F4AC996" Ref="Q?"  Part="1"
+AR Path="/60C74F5D/5F4AC996" Ref="Q?"  Part="1"
+AR Path="/60C9EA3E/5F4AC996" Ref="Q?"  Part="1"
 F 0 "Q?" V 5250 3850 50  0000 L CNN
 F 1 "BC857BS" V 5550 3850 50  0000 L CNN
@@
 U 2 1 6298DD74
 P 5850 4000
+AR Path="/60A4AB90/6298DD74" Ref="Q?"  Part="2"
+AR Path="/60C25BC1/6298DD74" Ref="Q?"  Part="2"
+AR Path="/60C51AC9/6298DD74" Ref="Q?"  Part="2"
+AR Path="/60C74F5D/6298DD74" Ref="Q?"  Part="2"
+AR Path="/60C9EA3E/6298DD74" Ref="Q?"  Part="2"
 F 0 "Q?" V 5750 3850 50  0000 L CNN
 F 1 "BC857BS" V 6050 3850 50  0000 L CNN
@@
 $Comp
 L mypartsLib:IRFHM9331PbF Q?
-U 1 1 5FB13230
+U 1 1 6051F954
 P 5600 3750
+AR Path="/60A4AB90/6051F954" Ref="Q?"  Part="1"
+AR Path="/60C25BC1/6051F954" Ref="Q?"  Part="1"
+AR Path="/60C51AC9/6051F954" Ref="Q?"  Part="1"
+AR Path="/60C74F5D/6051F954" Ref="Q?"  Part="1"
+AR Path="/60C9EA3E/6051F954" Ref="Q?"  Part="1"
 F 0 "Q?" V 5800 3750 50  0000 C CNN
 F 1 "IRFHM9331PbF" V 5900 3750 50  0000 C CNN
@@
 U 1 1 62DD7D73
 P 5400 4450
+AR Path="/60A4AB90/62DD7D73" Ref="R?"  Part="1"
+AR Path="/60C25BC1/62DD7D73" Ref="R?"  Part="1"
+AR Path="/60C51AC9/62DD7D73" Ref="R?"  Part="1"
+AR Path="/60C74F5D/62DD7D73" Ref="R?"  Part="1"
+AR Path="/60C9EA3E/62DD7D73" Ref="R?"  Part="1"
 F 0 "R?" V 5300 4350 50  0000 L CNN
 F 1 "1M" V 5400 4400 50  0000 L CNN
@@
 U 1 1 6253EB6F
 P 6300 3650
+AR Path="/60A4AB90/6253EB6F" Ref="TP?"  Part="1"
+AR Path="/60C25BC1/6253EB6F" Ref="TP?"  Part="1"
+AR Path="/60C51AC9/6253EB6F" Ref="TP?"  Part="1"
+AR Path="/60C74F5D/6253EB6F" Ref="TP?"  Part="1"
+AR Path="/60C9EA3E/6253EB6F" Ref="TP?"  Part="1"
 F 0 "TP?" V 6300 3800 50  0000 L CNN
 F 1 "TestPoint" V 6300 3850 50  0001 L CNN
@@
 U 1 1 6253E3D7
 P 4900 3650
+AR Path="/60A4AB90/6253E3D7" Ref="TP?"  Part="1"
+AR Path="/60C25BC1/6253E3D7" Ref="TP?"  Part="1"
+AR Path="/60C51AC9/6253E3D7" Ref="TP?"  Part="1"
+AR Path="/60C74F5D/6253E3D7" Ref="TP?"  Part="1"
+AR Path="/60C9EA3E/6253E3D7" Ref="TP?"  Part="1"
 F 0 "TP?" V 4900 3800 50  0000 L CNN
 F 1 "TestPoint" V 4900 3850 50  0001 L CNN
@@
 U 1 1 62DD8487
 P 5800 4450
+AR Path="/60A4AB90/62DD8487" Ref="R?"  Part="1"
+AR Path="/60C25BC1/62DD8487" Ref="R?"  Part="1"
+AR Path="/60C51AC9/62DD8487" Ref="R?"  Part="1"
+AR Path="/60C74F5D/62DD8487" Ref="R?"  Part="1"
+AR Path="/60C9EA3E/62DD8487" Ref="R?"  Part="1"
 F 0 "R?" V 5900 4350 50  0000 L CNN
 F 1 "1M" V 5800 4400 50  0000 L CNN
